Commit message: wow

File: urdf/dku_robotarm.urdf (robot description, URDF)
Before this commit: robot robotic_arm_6dof, 7 links, 6 joints
Links:
- added link main_gripper1, mass 11.975281293019925; collision mesh filename=package://dku_robotarm/meshes/main_gripper1.stl scale=0.001 0.001 0.001; visual mesh filename=package://dku_robotarm/meshes/main_gripper1.stl scale=0.001 0.001 0.001
- added link main_gripper2, mass 14.367402646416181; collision mesh filename=package://dku_robotarm/meshes/main_gripper2.stl scale=0.001 0.001 0.001; visual mesh filename=package://dku_robotarm/meshes/main_gripper2.stl scale=0.001 0.001 0.001
- added link sub_gripper1, mass 12.566774937192251; collision mesh filename=package://dku_robotarm/meshes/sub_gripper1.stl scale=0.001 0.001 0.001; visual mesh filename=package://dku_robotarm/meshes/sub_gripper1.stl scale=0.001 0.001 0.001
- added link sub_gripper2, mass 14.367402725616657; collision mesh filename=package://dku_robotarm/meshes/sub_gripper2.stl scale=0.001 0.001 0.001; visual mesh filename=package://dku_robotarm/meshes/sub_gripper2.stl scale=0.001 0.001 0.001
- link link5: mass 330.4055669252865 -> 262.6198877301529
Joints:
- added joint main_gripper1: type revolute, parent link5, child main_gripper1, origin xyz=-0.04646024 0.2879688399999986 0.15641769000000127 rpy=1.5707963267948966 -4.462142461080891e-15 1.5707963267948966, axis 0.0 -0.012509000000000027 -0.9999220000000002, limit lower=-1.570796 upper=1.570796 effort=1000000 velocity=1000000
- added joint main_gripper2: type revolute, parent main_gripper1, child main_gripper2, origin xyz=0.3076185800000002 -0.00032522999999994083 -0.025997959999999997 rpy=-1.734723475976844e-18 -2.5243548967072372e-29 6.037595893715346e-46, axis -2.5241579970252946e-29 -0.012509000000000025 -0.9999220000000002, limit lower=-1.570796 upper=1.570796 effort=1000000 velocity=1000000
- added joint sub_gripper1: type revolute, parent link5, child sub_gripper1, origin xyz=-0.00346603 0.2900000000000006 -0.12265295999999871 rpy=1.5707963267948966 -4.462142461080891e-15 1.5707963267948966, axis 0.0 -0.012509000000000027 -0.9999220000000002, limit lower=-1.570796 upper=1.570796 effort=1000000 velocity=1000000
- added joint sub_gripper2: type revolute, parent sub_gripper1, child sub_gripper2, origin xyz=0.30483807999999957 -0.04201389 -0.05947910999999998 rpy=-1.7347234759768194e-18 -2.5243548967072372e-29 6.0375958937149105e-46, axis -2.5241579970252946e-29 -0.012509000000000025 -0.9999220000000002, limit lower=-1.570796 upper=1.570796 effort=1000000 velocity=1000000
- joint base_joint: axis 1.5777218104420236e-30 -9.629638507136242e-16 1.0 -> 0.0 -9.62963850713621e-16 1.0; origin xyz=0.3232552899999969 -0.10588035999994976 1.249957100000006 rpy=-1.75011923755963e-14 -1.056843376502257e-14 9.142014000100513e-14 -> xyz=0.32325529000000003 -0.10588036 1.2499571 rpy=-9.62963850713621e-16 -0.0 0.0
- joint link1_link2: axis 1.26869229813338e-29 2.554632158605991e-15 -1.0 -> 0.012509 2.5544328972976203e-15 -0.9999220000000001; origin xyz=0.015010000000000403 -0.2675000000000001 0.14999999999999986 rpy=1.570796326794895 1.578492182419779e-30 -3.331398502653572e-31 -> xyz=0.01166272000000042 -0.26766683000000013 0.14999999999999986 rpy=1.570796326794895 -6.3108872417680615e-30 -3.398971393601724e-29
- joint link2_link3: axis -4.1797284106844794e-30 2.3946249947807627e-15 1.0 -> 0.012509 2.3944382140311698e-15 0.9999219999999999; origin xyz=0.0 1.03 2.6290081223123707e-15 rpy=-3.1415926535897882 -1.686665139201828e-29 2.5422275265868423e-32 -> xyz=0.0 1.03 2.6290081223123707e-15 rpy=-3.1415926535897882 6.322045984118727e-29 -6.3108872417679326e-30
- joint link3_link4: axis 6.728105408153287e-32 -3.3853306316112125e-15 1.0 -> 0.012509 -3.385066575821944e-15 0.999922; origin xyz=-0.015000000000000284 -0.9649900000000002 -0.022499999999997727 rpy=-5.779955626391975e-15 -4.2470094647660125e-30 2.542227526592168e-32 -> xyz=-0.01528028000000031 -0.9649900000000002 -0.022310609999997694 rpy=-5.779955626391973e-15 7.177747304298343e-29 -1.7188013101093054e-43
- joint link4_link5: axis 4.577930333900981e-30 0.9999999999999999 4.462142461080889e-15 -> 1.7347234760422044e-18 1.0 4.462142461080891e-15; origin xyz=-0.2700000000000013 -0.5774900000000014 0.34748999999999813 rpy=3.1415926535897922 4.262915079339174e-32 -4.578700705878737e-30 -> xyz=-0.2656321800000013 -0.5774900000000014 0.35084018999999805 rpy=3.1415926535897922 -4.096313271485057e-29 -1.7347234760422044e-18

Commit message: modify..

File: urdf/dku_robotarm.urdf (robot description, URDF)
Before this commit: robot robotic_arm_6dof, 11 links, 10 joints
Joints:
- joint end_effector: origin xyz=0 1.1 0 rpy=0.0 0.0 0.0 -> xyz=0 1.1 -0.01 rpy=0.0 0.0 0.0

Commit message: sdd

File: urdf/dku_robotarm.urdf (robot description, URDF)
Before this commit: robot robotic_arm_6dof, 11 links, 10 joints
Joints:
- joint end_effector: limit lower=-1.57 upper=1.57 effort=0.92 velocity=5.24 -> (none); type revolute -> fixed

Commit message: modify axis

File: urdf/dku_robotarm.urdf (robot description, URDF)
Before this commit: robot robotic_arm_6dof, 11 links, 10 joints
Links:
- link link1: mass 306.57866664253083 -> 306.5786666425041
- link link2: mass 100.44717038799456 -> 100.44717277373952
- link link3: mass 326.3184161312811 -> 326.31842277225974
Joints:
- joint base_joint: axis 0.0 -9.62963850713621e-16 1.0 -> 0.0 3.0656538569228853e-15 1.0; limit lower=-1.570796 upper=1.570796 effort=1000000 velocity=1000000 -> lower=-1.584512 upper=1.55708 effort=1000000 velocity=1000000; origin xyz=0.32325529000000003 -0.10588036 1.2499571 rpy=-9.62963850713621e-16 -0.0 0.0 -> xyz=0.10588036 0.32325529000000003 1.2519571 rpy=3.0656538569228853e-15 -0.0 0.0
- joint end_effector: origin xyz=0 1.1 -0.01 rpy=0.0 0.0 0.0 -> xyz=0.01 -1.1 0.01 rpy=0.0 0.0 0.0
- joint link1_link2: axis 0.012509 2.5544328972976203e-15 -0.9999220000000001 -> -0.9999059999999999 -3.5039334687439777e-17 0.013716000000006246; limit lower=-1.570796 upper=1.570796 effort=1000000 velocity=1000000 -> lower=-1.568677 upper=1.572916 effort=1000000 velocity=1000000; origin xyz=0.01166272000000042 -0.26766683000000013 0.14999999999999986 rpy=1.570796326794895 -6.3108872417680615e-30 -3.398971393601724e-29 -> xyz=0.26726897000000016 0.01867753000000043 0.14999999999999972 rpy=1.570796326794891 -1.039256748674529e-31 -1.734723475977927e-18
- joint link2_link3: axis 0.012509 2.3944382140311698e-15 0.9999219999999999 -> -9.352162046422787e-21 0.013715999999990076 -0.999906; limit lower=-1.570796 upper=1.570796 effort=1000000 velocity=1000000 -> lower=-1.570514 upper=1.571078 effort=1000000 velocity=1000000; origin xyz=0.0 1.03 2.6290081223123707e-15 rpy=-3.1415926535897882 6.322045984118727e-29 -6.3108872417679326e-30 -> xyz=2.993999999993946e-05 1.02999769 0.002182960000002652 rpy=1.5707963267949066 -2.5537647968680023e-15 1.5707963267948966
- joint link3_link4: axis 0.012509 -3.385066575821944e-15 0.999922 -> -0.999906 -4.686685962499137e-17 -0.013715999999996302; limit lower=-1.570796 upper=1.570796 effort=1000000 velocity=1000000 -> lower=-1.577655 upper=1.563938 effort=1000000 velocity=1000000; origin xyz=-0.01528028000000031 -0.9649900000000002 -0.022310609999997694 rpy=-5.779955626391973e-15 7.177747304298343e-29 -1.7188013101093054e-43 -> xyz=0.9649511900000005 0.0170072500000002 0.022735409999999873 rpy=1.5707963267949 -1.5707963267948855 0
- joint link4_link5: axis 1.7347234760422044e-18 1.0 4.462142461080891e-15 -> -6.100000000000043e-05 -0.9999900000000003 0.004455999999995753; origin xyz=-0.2656321800000013 -0.5774900000000014 0.35084018999999805 rpy=3.1415926535897922 -4.096313271485057e-29 -1.7347234760422044e-18 -> xyz=-0.343789430000001 -0.5786875400000008 -0.2721646099999981 rpy=-7.631778384881335e-15 1.8602830338647298e-19 4.2471464551046585e-19
- joint main_gripper1: axis 0.0 -0.012509000000000027 -0.9999220000000002 -> -0.004457 -0.999896 -0.013715999999999983; limit lower=-1.570796 upper=1.570796 effort=1000000 velocity=1000000 -> lower=-1.570796 upper=0.0 effort=1000000 velocity=1000000; origin xyz=-0.04646024 0.2879688399999986 0.15641769000000127 rpy=1.5707963267948966 -4.462142461080891e-15 1.5707963267948966 -> xyz=-0.1575997900000001 -0.28776766000000065 0.04362542999999879 rpy=-1.5707963267948966 4.246440975279546e-15 -1.5707963267948966
- joint main_gripper2: axis -2.5241579970252946e-29 -0.012509000000000025 -0.9999220000000002 -> -0.004457 -0.999896 -0.013715999999999978; limit lower=-1.570796 upper=1.570796 effort=1000000 velocity=1000000 -> (none); origin xyz=0.3076185800000002 -0.00032522999999994083 -0.025997959999999997 rpy=-1.734723475976844e-18 -2.5243548967072372e-29 6.037595893715346e-46 -> xyz=0.30749964999999974 -0.02736808 -0.0003754099999999916 rpy=-9.330926015963404e-19 -0.0 1.8663967412030045e-21; type revolute -> continuous
- joint sub_gripper1: axis 0.0 -0.012509000000000027 -0.9999220000000002 -> -0.004457 -0.999896 -0.013715999999999973; limit lower=-1.570796 upper=1.570796 effort=1000000 velocity=1000000 -> (none); origin xyz=-0.00346603 0.2900000000000006 -0.12265295999999871 rpy=1.5707963267948966 -4.462142461080891e-15 1.5707963267948966 -> xyz=0.12250216999999997 -0.2899748299999999 0.007973299999998771 rpy=-1.5707963267948966 4.246440975279546e-15 -1.5707963267948966; type revolute -> continuous
- joint sub_gripper2: axis -2.5241579970252946e-29 -0.012509000000000025 -0.9999220000000002 -> -0.004457 -0.999896 -0.013715999999999978; limit lower=-1.570796 upper=1.570796 effort=1000000 velocity=1000000 -> (none); origin xyz=0.30483807999999957 -0.04201389 -0.05947910999999998 rpy=-1.7347234759768194e-18 -2.5243548967072372e-29 6.0375958937149105e-46 -> xyz=0.30456767000000073 -0.06191816000000001 0.040421150000000024 rpy=-1.0251691368420165e-18 -8.673617379884035e-19 3.932017107160776e-21; type revolute -> continuous

Commit message: ddd

File: urdf/dku_robotarm.urdf (robot description, URDF)
Before this commit: robot robotic_arm_6dof, 11 links, 10 joints
Joints:
- joint link4_link5: limit lower=0.0 upper=3.141593 effort=1000000 velocity=1000000 -> lower=-1.570796 upper=1.570796 effort=1000000 velocity=1000000
- joint main_gripper1: axis -0.004457 -0.999896 -0.013715999999999983 -> -1.0441198370741651e-20 0.013715999999999978 -0.999906; origin xyz=-0.1575997900000001 -0.28776766000000065 0.04362542999999879 rpy=-1.5707963267948966 4.246440975279546e-15 -1.5707963267948966 -> xyz=-0.04236056999999972 -0.2936655399999995 -0.15627513000000126 rpy=-1.5707963267948966 4.2464459612885334e-15 -1.5707963267948966
- joint main_gripper2: axis -0.004457 -0.999896 -0.013715999999999978 -> -2.8919093855802717e-20 0.013715999999999978 -0.999906; origin xyz=0.30749964999999974 -0.02736808 -0.0003754099999999916 rpy=-9.330926015963404e-19 -0.0 1.8663967412030045e-21 -> xyz=0.3076155299999999 -0.0010141800000000067 -0.02601635 rpy=-5.157061093467415e-19 -6.581780574186106e-21 -8.673617379884034e-19
- joint sub_gripper1: axis -0.004457 -0.999896 -0.013715999999999973 -> -1.0441198370741651e-20 0.013715999999999978 -0.999906; origin xyz=0.12250216999999997 -0.2899748299999999 0.007973299999998771 rpy=-1.5707963267948966 4.246440975279546e-15 -1.5707963267948966 -> xyz=-0.006699080000000226 -0.29445069000000046 0.12383322999999877 rpy=-1.5707963267948966 4.2464459612885334e-15 -1.5707963267948966
- joint sub_gripper2: axis -0.004457 -0.999896 -0.013715999999999978 -> -4.2401764664552925e-21 0.013715999999999975 -0.999906; origin xyz=0.30456767000000073 -0.06191816000000001 0.040421150000000024 rpy=-1.0251691368420165e-18 -8.673617379884035e-19 3.932017107160776e-21 -> xyz=0.30465115000000026 -0.04179776999999998 -0.06057898 rpy=1.5641892085563873e-18 6.201604855142745e-21 -1.3835674616372782e-37
